Commit message: feat(script): add install script
Signed-off-by: m-brl <mathieu.borel@epitech.eu>

File: urdf/inmoov.urdf (robot description, URDF)
Before this commit: robot InMoov, 59 links, 58 joints
Links:
- link base_node: geometry visual mesh filename=package://inmoov_ros_sim/meshes/stl/stand.stl scale=1.00000 1.00000 1.00000
- link i01.head.eyeLeft_link: geometry visual mesh filename=package://inmoov_ros_sim/meshes/stl/Texture.011.stl scale=1.00000 1.00000 1.00000
- link i01.head.eyeRight_link: geometry visual mesh filename=package://inmoov_ros_sim/meshes/stl/Texture.012.stl scale=1.00000 1.00000 1.00000
- link i01.head.jaw_link: geometry visual mesh filename=package://inmoov_ros_sim/meshes/stl/Texture.014.stl scale=1.00000 1.00000 1.00000; visual mesh filename=package://inmoov_ros_sim/meshes/stl/Texture.086.stl scale=1.00000 1.00000 1.00000
- link i01.head.rothead_link: geometry visual mesh filename=package://inmoov_ros_sim/meshes/stl/Texture.013.stl scale=1.00000 1.00000 1.00000; visual mesh filename=package://inmoov_ros_sim/meshes/stl/Texture.068.stl scale=1.00000 1.00000 1.00000
- link i01.leftHand.index2_link: geometry visual mesh filename=package://inmoov_ros_sim/meshes/stl/Texture.019.stl scale=1.00000 1.00000 1.00000
- link i01.leftHand.index3_link: geometry visual mesh filename=package://inmoov_ros_sim/meshes/stl/Texture.020.stl scale=1.00000 1.00000 1.00000
- link i01.leftHand.index_link: geometry visual mesh filename=package://inmoov_ros_sim/meshes/stl/Texture.018.stl scale=1.00000 1.00000 1.00000
- link i01.leftHand.majeure2_link: geometry visual mesh filename=package://inmoov_ros_sim/meshes/stl/Texture.023.stl scale=1.00000 1.00000 1.00000
- link i01.leftHand.majeure3_link: geometry visual mesh filename=package://inmoov_ros_sim/meshes/stl/Texture.024.stl scale=1.00000 1.00000 1.00000
- link i01.leftHand.majeure_link: geometry visual mesh filename=package://inmoov_ros_sim/meshes/stl/Texture.022.stl scale=1.00000 1.00000 1.00000
- link i01.leftHand.pinky0_link: geometry visual mesh filename=package://inmoov_ros_sim/meshes/stl/Texture.041.stl scale=1.00000 1.00000 1.00000
- link i01.leftHand.pinky2_link: geometry visual mesh filename=package://inmoov_ros_sim/meshes/stl/Texture.028.stl scale=1.00000 1.00000 1.00000
- link i01.leftHand.pinky3_link: geometry visual mesh filename=package://inmoov_ros_sim/meshes/stl/Texture.029.stl scale=1.00000 1.00000 1.00000
- link i01.leftHand.pinky_link: geometry visual mesh filename=package://inmoov_ros_sim/meshes/stl/Texture.027.stl scale=1.00000 1.00000 1.00000
- link i01.leftHand.ringFinger_link: geometry visual mesh filename=package://inmoov_ros_sim/meshes/stl/Texture.032.stl scale=1.00000 1.00000 1.00000
- link i01.leftHand.ringfinger0_link: geometry visual mesh filename=package://inmoov_ros_sim/meshes/stl/Texture.040.stl scale=1.00000 1.00000 1.00000
- link i01.leftHand.ringfinger2_link: geometry visual mesh filename=package://inmoov_ros_sim/meshes/stl/Texture.033.stl scale=1.00000 1.00000 1.00000
- link i01.leftHand.ringfinger3_link: geometry visual mesh filename=package://inmoov_ros_sim/meshes/stl/Texture.034.stl scale=1.00000 1.00000 1.00000
- link i01.leftHand.thumb1_link: geometry visual mesh filename=package://inmoov_ros_sim/meshes/stl/Texture.035.stl scale=1.00000 1.00000 1.00000
- link i01.leftHand.thumb3_link: geometry visual mesh filename=package://inmoov_ros_sim/meshes/stl/Texture.038.stl scale=1.00000 1.00000 1.00000
- link i01.leftHand.thumb_link: geometry visual mesh filename=package://inmoov_ros_sim/meshes/stl/Texture.037.stl scale=1.00000 1.00000 1.00000
- link i01.leftHand.wrist.001_link: geometry visual mesh filename=package://inmoov_ros_sim/meshes/stl/Texture.235.stl scale=1.00000 1.00000 1.00000
- link i01.rightHand.index2_link: geometry visual mesh filename=package://inmoov_ros_sim/meshes/stl/Texture.045.stl scale=1.00000 1.00000 1.00000
- link i01.rightHand.index3_link: geometry visual mesh filename=package://inmoov_ros_sim/meshes/stl/Texture.046.stl scale=1.00000 1.00000 1.00000
- link i01.rightHand.index_link: geometry visual mesh filename=package://inmoov_ros_sim/meshes/stl/Texture.044.stl scale=1.00000 1.00000 1.00000
- link i01.rightHand.majeure2_link: geometry visual mesh filename=package://inmoov_ros_sim/meshes/stl/Texture.049.stl scale=1.00000 1.00000 1.00000
- link i01.rightHand.majeure3_link: geometry visual mesh filename=package://inmoov_ros_sim/meshes/stl/Texture.050.stl scale=1.00000 1.00000 1.00000
- link i01.rightHand.majeure_link: geometry visual mesh filename=package://inmoov_ros_sim/meshes/stl/Texture.048.stl scale=1.00000 1.00000 1.00000
- link i01.rightHand.pinky0_link: geometry visual mesh filename=package://inmoov_ros_sim/meshes/stl/Texture.067.stl scale=1.00000 1.00000 1.00000
- link i01.rightHand.pinky2_link: geometry visual mesh filename=package://inmoov_ros_sim/meshes/stl/Texture.054.stl scale=1.00000 1.00000 1.00000
- link i01.rightHand.pinky3_link: geometry visual mesh filename=package://inmoov_ros_sim/meshes/stl/Texture.055.stl scale=1.00000 1.00000 1.00000
- link i01.rightHand.pinky_link: geometry visual mesh filename=package://inmoov_ros_sim/meshes/stl/Texture.053.stl scale=1.00000 1.00000 1.00000
- link i01.rightHand.ringFinger_link: geometry visual mesh filename=package://inmoov_ros_sim/meshes/stl/Texture.058.stl scale=1.00000 1.00000 1.00000
- link i01.rightHand.ringfinger0_link: geometry visual mesh filename=package://inmoov_ros_sim/meshes/stl/Texture.066.stl scale=1.00000 1.00000 1.00000
- link i01.rightHand.ringfinger2_link: geometry visual mesh filename=package://inmoov_ros_sim/meshes/stl/Texture.059.stl scale=1.00000 1.00000 1.00000
- link i01.rightHand.ringfinger3_link: geometry visual mesh filename=package://inmoov_ros_sim/meshes/stl/Texture.060.stl scale=1.00000 1.00000 1.00000
- link i01.rightHand.thumb1_link: geometry visual mesh filename=package://inmoov_ros_sim/meshes/stl/Texture.063.stl scale=1.00000 1.00000 1.00000
- link i01.rightHand.thumb3_link: geometry visual mesh filename=package://inmoov_ros_sim/meshes/stl/Texture.062.stl scale=1.00000 1.00000 1.00000
- link i01.rightHand.thumb_link: geometry visual mesh filename=package://inmoov_ros_sim/meshes/stl/Texture.061.stl scale=1.00000 1.00000 1.00000
- link i01.rightHand.wrist.001_link: geometry visual mesh filename=package://inmoov_ros_sim/meshes/stl/Texture.204.stl scale=1.00000 1.00000 1.00000
- link left_elbow_x_link: geometry visual mesh filename=package://inmoov_ros_sim/meshes/stl/Texture.007.stl scale=1.00000 1.00000 1.00000; visual mesh filename=package://inmoov_ros_sim/meshes/stl/Texture.236.stl scale=1.00000 1.00000 1.00000
- link left_shoulder_x_link: geometry visual mesh filename=package://inmoov_ros_sim/meshes/stl/Texture.003.stl scale=1.00000 1.00000 1.00000; visual mesh filename=package://inmoov_ros_sim/meshes/stl/Texture.254.stl scale=1.00000 1.00000 1.00000
- link left_shoulder_y_link: geometry visual mesh filename=package://inmoov_ros_sim/meshes/stl/Texture.004.stl scale=1.00000 1.00000 1.00000; visual mesh filename=package://inmoov_ros_sim/meshes/stl/Texture.248.stl scale=1.00000 1.00000 1.00000
- link left_shoulder_z_link: geometry visual mesh filename=package://inmoov_ros_sim/meshes/stl/G-__564753.001.stl scale=1.00000 1.00000 1.00000; visual mesh filename=package://inmoov_ros_sim/meshes/stl/G-__564753.002.stl scale=1.00000 1.00000 1.00000
- link left_wrist_z_link: geometry visual mesh filename=package://inmoov_ros_sim/meshes/stl/Texture.039.stl scale=1.00000 1.00000 1.00000
- link neck_link: geometry visual mesh filename=package://inmoov_ros_sim/meshes/stl/Texture.015.stl scale=1.00000 1.00000 1.00000; visual mesh filename=package://inmoov_ros_sim/meshes/stl/Texture.083.stl scale=1.00000 1.00000 1.00000
- link right_elbow_x_link: geometry visual mesh filename=package://inmoov_ros_sim/meshes/stl/Texture.008.stl scale=1.00000 1.00000 1.00000; visual mesh filename=package://inmoov_ros_sim/meshes/stl/Texture.205.stl scale=1.00000 1.00000 1.00000
- link right_shoulder_x_link: geometry visual mesh filename=package://inmoov_ros_sim/meshes/stl/Texture.005.stl scale=1.00000 1.00000 1.00000; visual mesh filename=package://inmoov_ros_sim/meshes/stl/Texture.223.stl scale=1.00000 1.00000 1.00000
- link right_shoulder_y_link: geometry visual mesh filename=package://inmoov_ros_sim/meshes/stl/Texture.006.stl scale=1.00000 1.00000 1.00000; visual mesh filename=package://inmoov_ros_sim/meshes/stl/Texture.217.stl scale=1.00000 1.00000 1.00000
- link right_shoulder_z_link: geometry visual mesh filename=package://inmoov_ros_sim/meshes/stl/G-__566220.001.stl scale=1.00000 1.00000 1.00000; visual mesh filename=package://inmoov_ros_sim/meshes/stl/G-__566220.002.stl scale=1.00000 1.00000 1.00000
- link right_wrist_z_link: geometry visual mesh filename=package://inmoov_ros_sim/meshes/stl/Texture.065.stl scale=1.00000 1.00000 1.00000
- link torso_bottom_link: geometry visual mesh filename=package://inmoov_ros_sim/meshes/stl/Texture.002.stl scale=1.00000 1.00000 1.00000; visual mesh filename=package://inmoov_ros_sim/meshes/stl/Texture.195.stl scale=1.00000 1.00000 1.00000
- link torso_y_link: geometry visual mesh filename=package://inmoov_ros_sim/meshes/stl/Texture.088.stl scale=1.00000 1.00000 1.00000; visual mesh filename=package://inmoov_ros_sim/meshes/stl/Texture.089.stl scale=1.00000 1.00000 1.00000
- link torso_z_link: geometry visual mesh filename=package://inmoov_ros_sim/meshes/stl/Texture.001.stl scale=1.00000 1.00000 1.00000; visual mesh filename=package://inmoov_ros_sim/meshes/stl/Texture.167.stl scale=1.00000 1.00000 1.00000
